File: _autosave-pcb.sch (KiCad schematic (older format))
At the start: 14 parts

Commit message: addtypec
Parts:
- added F?: 500mA, Fuse_Holders_and_Fuses:Fuse_SMD1206_Reflow, symbol Device:Polyfuse_Small
- added R? (x2): 22, Resistors_SMD:R_0805, symbol Device:R_Small
- added R? (x2): 5.1k, Resistors_SMD:R_0805, symbol Device:R_Small
- added U?: PRTR5V0U2X, locallib:SOT143B, symbol ai03-locallib:PRTR5V0U2X
- added USB?: HRO-TYPE-C-31-M-12, Type-C:HRO-TYPE-C-31-M-12-Assembly, symbol Type-C:HRO-TYPE-C-31-M-12
Connections:
- net labels added: VCC
- wire segments 46 -> 89
Other:
- moved on the sheet: C?, R?, SW?, U?, Y?
